File: ModuCard-GPIO-AUX/HalfBridge.kicad_sch (KiCad schematic)
At the start: 33 parts, among them Q1 XR30N06F, Q2 XR30N06F, U1 DGD0506AM10-13

Commit message: wip
Parts:
- removed C10, C11, C12, C13, C14, C15, C16, C17, C18, C19, C20, C21, C6, C7, C8, C9: 10uF, PCM_JLCPCB:C_0805, symbol PCM_JLCPCB-Capacitors:0805,10uF,(2)
- added R62: 10kΩ, PCM_JLCPCB:R_0603x4, symbol PCM_JLCPCB-Resistors:0603x4,10kΩ
Connections:
- net GND: now also R62.6, R62.7
- net VIN_BRIDGE: now also R62.1, R62.4
- net at C4.2, C5.1: now also R62.3, R62.5
- net at C2.2, C3.1: now also R62.2, R62.8
- net at U1.10 (LO): now also R7.1
- net at U1.5 (NC): no longer R7.1
Other:
- moved on the sheet: C2, C3, C4, C5
