File: ModuCard-GPIO-AUX/ModuCard-GPIO-AUX.kicad_sch (KiCad schematic)
At the start: 0 parts

Commit message: wip
Changed lines of the file:
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@@
 	(generator_version "9.0")
 	(paper "A4")
-	(sheet
-		(at 139.7 44.45)
+	(bus
+		(pts
+			(xy 151.13 66.04) (xy 170.18 66.04)
+		)
+		(stroke
+			(width 0)
+			(type default)
+		)
+	)
+	(bus
+		(pts
+			(xy 151.13 66.04) (xy 151.13 80.01)
+		)
+		(stroke
+			(width 0)
+			(type default)
+		)
+	)
+	(sheet
+		(at 170.18 43.18)
 		(size 36.83 10.16)
 		(exclude_from_sim no)
@@
 		)
 		(property "Sheetname" "PowerIN"
-			(at 139.7 43.7384 0)
+			(at 170.18 42.4684 0)
 			(effects
 				(font
@@
 		)
 		(property "Sheetfile" "PowerIN.kicad_sch"
-			(at 139.7 55.1946 0)
+			(at 170.18 53.9246 0)
 			(effects
 				(font
@@
 	)
 	(sheet
-		(at 52.07 63.5)
+		(at 62.23 63.5)
 		(size 36.83 48.26)
 		(exclude_from_sim no)
@@
 		)
 		(property "Sheetname" "backplane"
-			(at 52.07 62.7884 0)
+			(at 62.23 62.7884 0)
 			(effects
 				(font
@@
 		)
 		(property "Sheetfile" "backplane.kicad_sch"
-			(at 52.07 112.3446 0)
+			(at 62.23 112.3446 0)
 			(effects
 				(font
@@
 		)
 		(pin "GPIOC[0..15]" input
-			(at 88.9 68.58 0)
+			(at 99.06 68.58 0)
 			(effects
 				(font
@@
 		)
 		(pin "BACKPLANE{USB}" output
-			(at 88.9 85.09 0)
+			(at 99.06 85.09 0)
 			(effects
 				(font
@@
 		)
 		(pin "CAN2{CAN}" bidirectional
-			(at 88.9 100.33 0)
+			(at 99.06 100.33 0)
 			(effects
 				(font
@@
 		)
 		(pin "GPIOR[0..15]" input
-			(at 88.9 71.12 0)
+			(at 99.06 71.12 0)
 			(effects
 				(font
@@
 		)
 		(pin "CAN1{CAN}" bidirectional
-			(at 88.9 102.87 0)
+			(at 99.06 102.87 0)
 			(effects
 				(font
@@
 		)
 		(pin "GPIOL[0..15]" input
-			(at 88.9 73.66 0)
+			(at 99.06 73.66 0)
 			(effects
 				(font
@@
 	)
 	(sheet
-		(at 139.7 105.41)
+		(at 170.18 104.14)
 		(size 35.56 7.62)
 		(exclude_from_sim no)
@@
 		)
 		(property "Sheetname" "Conn4"
-			(at 139.7 104.6984 0)
-			(effects
-				(font
-					(size 1.27 1.27)
-				)
-				(justify left bottom)
-			)
-		)
-		(property "Sheetfile" "Conn1.kicad_sch"
-			(at 139.7 113.6146 0)
-			(effects
-				(font
-					(size 1.27 1.27)
-				)
-				(justify left top)
-			)
-		)
-		(pin "GPIO" input
-			(at 139.7 109.22 180)
+			(at 170.18 103.4284 0)
+			(effects
+				(font
+					(size 1.27 1.27)
+				)
+				(justify left bottom)
+			)
+		)
+		(property "Sheetfile" "Conn1.kicad_sch"
+			(at 170.18 112.3446 0)
+			(effects
+				(font
+					(size 1.27 1.27)
+				)
+				(justify left top)
+			)
+		)
+		(pin "GPIO" input
+			(at 170.18 107.95 180)
 			(effects
 				(font
@@
 	)
 	(sheet
-		(at 139.7 77.47)
+		(at 170.18 76.2)
 		(size 35.56 7.62)
 		(exclude_from_sim no)
@@
 		)
 		(property "Sheetname" "Conn2"
-			(at 139.7 76.7584 0)
-			(effects
-				(font
-					(size 1.27 1.27)
-				)
-				(justify left bottom)
-			)
-		)
-		(property "Sheetfile" "Conn1.kicad_sch"
-			(at 139.7 85.6746 0)
-			(effects
-				(font
-					(size 1.27 1.27)
-				)
-				(justify left top)
-			)
-		)
-		(pin "GPIO" input
-			(at 139.7 81.28 180)
+			(at 170.18 75.4884 0)
+			(effects
+				(font
+					(size 1.27 1.27)
+				)
+				(justify left bottom)
+			)
+		)
+		(property "Sheetfile" "Conn1.kicad_sch"
+			(at 170.18 84.4046 0)
+			(effects
+				(font
+					(size 1.27 1.27)
+				)
+				(justify left top)
+			)
+		)
+		(pin "GPIO" input
+			(at 170.18 80.01 180)
 			(effects
 				(font
@@
 	)
 	(sheet
-		(at 139.7 119.38)
+		(at 170.18 118.11)
 		(size 35.56 7.62)
 		(exclude_from_sim no)
@@
 		)
 		(property "Sheetname" "Conn5"
-			(at 139.7 118.6684 0)
-			(effects
-				(font
-					(size 1.27 1.27)
-				)
-				(justify left bottom)
-			)
-		)
-		(property "Sheetfile" "Conn1.kicad_sch"
-			(at 139.7 127.5846 0)
-			(effects
-				(font
-					(size 1.27 1.27)
-				)
-				(justify left top)
-			)
-		)
-		(pin "GPIO" input
-			(at 139.7 123.19 180)
+			(at 170.18 117.3984 0)
+			(effects
+				(font
+					(size 1.27 1.27)
+				)
+				(justify left bottom)
+			)
+		)
+		(property "Sheetfile" "Conn1.kicad_sch"
+			(at 170.18 126.3146 0)
+			(effects
+				(font
+					(size 1.27 1.27)
+				)
+				(justify left top)
+			)
+		)
+		(pin "GPIO" input
+			(at 170.18 121.92 180)
 			(effects
 				(font
@@
 	)
 	(sheet
-		(at 139.7 91.44)
+		(at 170.18 90.17)
 		(size 35.56 7.62)
 		(exclude_from_sim no)
@@
 		)
 		(property "Sheetname" "Conn3"
-			(at 139.7 90.7284 0)
-			(effects
-				(font
-					(size 1.27 1.27)
-				)
-				(justify left bottom)
-			)
-		)
-		(property "Sheetfile" "Conn1.kicad_sch"
-			(at 139.7 99.6446 0)
-			(effects
-				(font
-					(size 1.27 1.27)
-				)
-				(justify left top)
-			)
-		)
-		(pin "GPIO" input
-			(at 139.7 95.25 180)
+			(at 170.18 89.4584 0)
+			(effects
+				(font
+					(size 1.27 1.27)
+				)
+				(justify left bottom)
+			)
+		)
+		(property "Sheetfile" "Conn1.kicad_sch"
+			(at 170.18 98.3746 0)
+			(effects
+				(font
+					(size 1.27 1.27)
+				)
+				(justify left top)
+			)
+		)
+		(pin "GPIO" input
+			(at 170.18 93.98 180)
 			(effects
 				(font
@@
 	)
 	(sheet
-		(at 139.7 63.5)
+		(at 170.18 62.23)
 		(size 35.56 7.62)
 		(exclude_from_sim no)
@@
 		)
 		(property "Sheetname" "Conn1"
-			(at 139.7 62.7884 0)
-			(effects
-				(font
-					(size 1.27 1.27)
-				)
-				(justify left bottom)
-			)
-		)
-		(property "Sheetfile" "Conn1.kicad_sch"
-			(at 139.7 71.7046 0)
-			(effects
-				(font
-					(size 1.27 1.27)
-				)
-				(justify left top)
-			)
-		)
-		(pin "GPIO" input
-			(at 139.7 67.31 180)
-			(effects
-				(font
+			(at 170.18 61.5184 0)
+			(effects
+				(font
+					(size 1.27 1.27)
+				)
+				(justify left bottom)
+			)
+		)
+		(property "Sheetfile" "Conn1.kicad_sch"
+			(at 170.18 70.4346 0)
+			(effects
+				(font
+					(size 1.27 1.27)
+				)
+				(justify left top)
+			)
+		)
+		(pin "GPIO" input
+			(at 170.18 66.04 180)
+			(effects
+				(font
